File: HackRPI-Badge.brd (EAGLE design)
At the start: 124.5 x 94 mm, 42 parts, among them J1 FTDI_BASICPTH, J2 SOLDERJUMPERTRACE-PTH, U2 3.3V, U4 74595, U5 74595, U6 74595, U7 74165DT, U8 AT25FS010

Commit message: Added bom partno attributes to all parts
Parts:
- U8: value AT25FS010 -> AT25SF041
