File: eagle/HackRPI-Badge.brd (EAGLE design)
At the start: 118.1 x 76.2 mm, 43 parts, among them J1 FTDI_BASICPTH, J2 SOLDERJUMPERPTH, U2 3.3V, U4 74595, U5 74595, U6 74595, U7 74165DT

Commit message: Fixed LED matrix name typo, updated BOM info for a capacitor
Parts:
- renumbered LEF_RIGHT to LED_RIGHT
Changed lines of the file:
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@@
 <attribute name="PARTNO" value="LDM-13488MI" x="27.94" y="22.1" size="1.778" layer="27" rot="R90" display="off"/>
 </element>
-<element name="LEF_RIGHT" library="mylib" package="32MM_LEDMATRIX" value="8X8LEDMATRIX_COLUMN_CATHODELDM-13488MI" x="27.94" y="54.1" rot="R90">
+<element name="LED_RIGHT" library="mylib" package="32MM_LEDMATRIX" value="8X8LEDMATRIX_COLUMN_CATHODELDM-13488MI" x="27.94" y="54.1" rot="R90">
 <attribute name="PARTNO" value="LDM-13488MI" x="27.94" y="54.1" size="1.778" layer="27" rot="R90" display="off"/>
 </element>
@@
 <attribute name="NAME" x="105.029" y="29.718" size="0.8128" layer="25" font="vector" rot="R180"/>
 <attribute name="VALUE" x="105.156" y="28.7655" size="0.4064" layer="27" font="vector" rot="R180"/>
+<attribute name="PARTNO" value="GRM155R61A105KE15D" x="104.14" y="27.6225" size="1.778" layer="27" rot="R180" display="off"/>
 </element>
 <element name="J2" library="SparkFun-Retired" package="SJ_2S-PTH" value="SOLDERJUMPERPTH" x="92.3925" y="68.58" rot="R90"/>
@@
 <signal name="N$7">
 <contactref element="LED_LEFT" pad="9"/>
-<contactref element="LEF_RIGHT" pad="9"/>
+<contactref element="LED_RIGHT" pad="9"/>
 <contactref element="U3" pad="18"/>
 <wire x1="33.53" y1="30.99" x2="37.975" y2="35.435" width="0.4064" layer="1"/>
@@
 </signal>
 <signal name="N$14">
-<contactref element="LEF_RIGHT" pad="14"/>
+<contactref element="LED_RIGHT" pad="14"/>
 <contactref element="LED_LEFT" pad="14"/>
 <contactref element="U3" pad="17"/>
@@
 <signal name="N$15">
 <contactref element="LED_LEFT" pad="8"/>
-<contactref element="LEF_RIGHT" pad="8"/>
+<contactref element="LED_RIGHT" pad="8"/>
 <contactref element="U3" pad="16"/>
 <wire x1="49.53" y1="43.0022" x2="49.53" y2="41.91" width="0.4064" layer="1"/>
@@
 </signal>
 <signal name="N$16">
-<contactref element="LEF_RIGHT" pad="12"/>
+<contactref element="LED_RIGHT" pad="12"/>
 <contactref element="LED_LEFT" pad="12"/>
 <contactref element="U3" pad="15"/>
@@
 <signal name="N$17">
 <contactref element="LED_LEFT" pad="1"/>
-<contactref element="LEF_RIGHT" pad="1"/>
+<contactref element="LED_RIGHT" pad="1"/>
 <contactref element="U3" pad="14"/>
 <wire x1="39.94" y1="13.21" x2="36.83" y2="16.32" width="0.4064" layer="16"/>
@@
 </signal>
 <signal name="N$18">
-<contactref element="LEF_RIGHT" pad="7"/>
+<contactref element="LED_RIGHT" pad="7"/>
 <contactref element="LED_LEFT" pad="7"/>
 <contactref element="U3" pad="13"/>
@@
 <signal name="N$19">
 <contactref element="LED_LEFT" pad="2"/>
-<contactref element="LEF_RIGHT" pad="2"/>
+<contactref element="LED_RIGHT" pad="2"/>
 <contactref element="U3" pad="12"/>
 <wire x1="39.94" y1="47.75" x2="53.215" y2="47.75" width="0.4064" layer="16"/>
@@
 </signal>
 <signal name="N$20">
-<contactref element="LEF_RIGHT" pad="5"/>
+<contactref element="LED_RIGHT" pad="5"/>
 <contactref element="LED_LEFT" pad="5"/>
 <contactref element="U3" pad="11"/>
@@
 <signal name="N$23">
 <contactref element="RN3" pad="1"/>
-<contactref element="LEF_RIGHT" pad="13"/>
+<contactref element="LED_RIGHT" pad="13"/>
 <wire x1="15.94" y1="52.83" x2="16.635" y2="52.83" width="0.4064" layer="16"/>
 <wire x1="16.635" y1="52.83" x2="19.05" y2="55.245" width="0.4064" layer="16"/>
@@
 <signal name="N$24">
 <contactref element="RN3" pad="2"/>
-<contactref element="LEF_RIGHT" pad="3"/>
+<contactref element="LED_RIGHT" pad="3"/>
 <wire x1="45.73" y1="56.28" x2="42.945" y2="56.28" width="0.4064" layer="1"/>
 <wire x1="42.945" y1="56.28" x2="41.91" y2="55.245" width="0.4064" layer="1"/>
@@
 <signal name="N$25">
 <contactref element="RN3" pad="3"/>
-<contactref element="LEF_RIGHT" pad="4"/>
+<contactref element="LED_RIGHT" pad="4"/>
 <wire x1="45.73" y1="55.48" x2="43.415" y2="55.48" width="0.4064" layer="1"/>
 <wire x1="43.415" y1="55.48" x2="43.18" y2="55.245" width="0.4064" layer="1"/>
@@
 <signal name="N$26">
 <contactref element="RN3" pad="4"/>
-<contactref element="LEF_RIGHT" pad="10"/>
+<contactref element="LED_RIGHT" pad="10"/>
 <wire x1="45.73" y1="54.68" x2="43.885" y2="54.68" width="0.4064" layer="1"/>
 <wire x1="43.885" y1="54.68" x2="43.18" y2="53.975" width="0.4064" layer="1"/>
@@
 <signal name="N$27">
 <contactref element="RN4" pad="1"/>
-<contactref element="LEF_RIGHT" pad="6"/>
+<contactref element="LED_RIGHT" pad="6"/>
 <wire x1="45.73" y1="53.27" x2="44.52" y2="53.27" width="0.4064" layer="1"/>
 <wire x1="44.52" y1="53.27" x2="44.45" y2="53.34" width="0.4064" layer="1"/>
@@
 <signal name="N$28">
 <contactref element="RN4" pad="2"/>
-<contactref element="LEF_RIGHT" pad="11"/>
+<contactref element="LED_RIGHT" pad="11"/>
 <wire x1="45.73" y1="52.47" x2="44.85" y2="52.47" width="0.4064" layer="1"/>
 <wire x1="44.85" y1="52.47" x2="43.18" y2="50.8" width="0.4064" layer="1"/>
@@
 <signal name="N$29">
 <contactref element="RN4" pad="3"/>
-<contactref element="LEF_RIGHT" pad="15"/>
+<contactref element="LED_RIGHT" pad="15"/>
 <wire x1="45.73" y1="51.67" x2="45.32" y2="51.67" width="0.4064" layer="1"/>
 <wire x1="45.32" y1="51.67" x2="44.45" y2="50.8" width="0.4064" layer="1"/>
@@
 <signal name="N$30">
 <contactref element="RN4" pad="4"/>
-<contactref element="LEF_RIGHT" pad="16"/>
+<contactref element="LED_RIGHT" pad="16"/>
 <wire x1="15.94" y1="45.21" x2="15.94" y2="39.94" width="0.4064" layer="1"/>
 <wire x1="15.94" y1="39.94" x2="17.78" y2="38.1" width="0.4064" layer="1"/>
